File: hardware/pawb_sao.kicad_pcb (KiCad board)
At the start: 2 copper layers, 40.4 x 40.6 mm, 33 parts, among them J1 PROG, J5 SAO, Q1 MMBT3904, SW1 GREEN, SW2 RED, SW3 YELLOW, SW4 BLUE, U2 CH32V003FxPx

Commit message: made 3d model
Parts:
- SW1, SW2, SW3, SW4: footprint Button_Switch_SMD:SW_SPST_EVQP0 -> pawb_sao:SW_SPST_EVQP0
- moved H2 3.19 mm to (184.7, 103.0)
Changed lines of the file:
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@@
 		(embedded_fonts no)
 	)
-	(footprint "Button_Switch_SMD:SW_SPST_EVQP0"
+	(footprint "pawb_sao:SW_SPST_EVQP0"
 		(layer "F.Cu")
 		(at 158.07 95.93 180)
@@
 			(at 0 -3.9 180)
 			(unlocked yes)
-			(layer "F.Fab")
-			(hide yes)
+			(layer "F.SilkS")
 			(effects
 				(font
@@
 			(unlocked yes)
 			(layer "F.Fab")
-			(hide yes)
 			(effects
 				(font
@@
 		)
 		(embedded_fonts no)
-		(model "${KICAD9_3DMODEL_DIR}/Button_Switch_SMD.3dshapes/SW_SPST_EVQP0.step"
+		(model "${KIPRJMOD}/3d/SON4_PTS526SM15SMTR2LFS_CNK.step"
 			(offset
 				(xyz 0 0 0)
@@
 		)
 	)
-	(footprint "Button_Switch_SMD:SW_SPST_EVQP0"
+	(footprint "pawb_sao:SW_SPST_EVQP0"
 		(layer "F.Cu")
 		(at 177.36 87.58 180)
@@
 			(at 0 -3.9 180)
 			(unlocked yes)
-			(layer "F.Fab")
-			(hide yes)
+			(layer "F.SilkS")
 			(effects
 				(font
@@
 			(unlocked yes)
 			(layer "F.Fab")
-			(hide yes)
 			(effects
 				(font
@@
 		)
 		(embedded_fonts no)
-		(model "${KICAD9_3DMODEL_DIR}/Button_Switch_SMD.3dshapes/SW_SPST_EVQP0.step"
+		(model "${KIPRJMOD}/3d/SON4_PTS526SM15SMTR2LFS_CNK.step"
 			(offset
 				(xyz 0 0 0)
@@
 		)
 		(embedded_fonts no)
+		(model "${KIPRJMOD}/3d/SMTB-0940-T-3V-R.STEP"
+			(offset
+				(xyz 0 0 1)
+			)
+			(scale
+				(xyz 1 1 1)
+			)
+			(rotate
+				(xyz -90 -0 90)
+			)
+		)
 	)
 	(footprint "Resistor_SMD:R_0402_1005Metric"
@@
 	(footprint "MountingHole:MountingHole_2.2mm_M2"
 		(layer "F.Cu")
-		(at 181.6 103.69)
+		(at 184.71 103)
 		(descr "Mounting Hole 2.2mm, M2, no annular, generated by kicad-footprint-generator mountinghole.py")
 		(tags "mountinghole M2")
@@
 		(embedded_fonts no)
 	)
-	(footprint "Button_Switch_SMD:SW_SPST_EVQP0"
+	(footprint "pawb_sao:SW_SPST_EVQP0"
 		(layer "F.Cu")
 		(at 165.9 87.73 180)
@@
 			(at 0 -3.9 180)
 			(unlocked yes)
-			(layer "F.Fab")
-			(hide yes)
+			(layer "F.SilkS")
 			(effects
 				(font
@@
 			(unlocked yes)
 			(layer "F.Fab")
-			(hide yes)
 			(effects
 				(font
@@
 		)
 		(embedded_fonts no)
-		(model "${KICAD9_3DMODEL_DIR}/Button_Switch_SMD.3dshapes/SW_SPST_EVQP0.step"
+		(model "${KIPRJMOD}/3d/SON4_PTS526SM15SMTR2LFS_CNK.step"
 			(offset
 				(xyz 0 0 0)
@@
 		)
 	)
-	(footprint "Button_Switch_SMD:SW_SPST_EVQP0"
+	(footprint "pawb_sao:SW_SPST_EVQP0"
 		(layer "F.Cu")
 		(at 186.17 95.38 180)
@@
 			(at 0 -3.9 180)
 			(unlocked yes)
-			(layer "F.Fab")
-			(hide yes)
+			(layer "F.SilkS")
 			(effects
 				(font
@@
 			(unlocked yes)
 			(layer "F.Fab")
-			(hide yes)
 			(effects
 				(font
@@
 		)
 		(embedded_fonts no)
-		(model "${KICAD9_3DMODEL_DIR}/Button_Switch_SMD.3dshapes/SW_SPST_EVQP0.step"
+		(model "${KIPRJMOD}/3d/SON4_PTS526SM15SMTR2LFS_CNK.step"
 			(offset
 				(xyz 0 0 0)
@@
 		)
 		(embedded_fonts no)
+		(model "${KIPRJMOD}/3d/bh-25f-1.stp"
+			(offset
+				(xyz 0 -110 2.7)
+			)
+			(scale
+				(xyz 1 1 1)
+			)
+			(rotate
+				(xyz -90 -0 90)
+			)
+		)
 	)
 	(footprint "TestPoint:TestPoint_Pad_D1.5mm"
@@
 	(gr_poly
 		(pts
-			(xy 186.25 101.185) (xy 185.25 102.185) (xy 184.25 101.185)
+			(xy 187.79 101.38) (xy 186.79 102.38) (xy 185.79 101.38)
 		)
 		(stroke
@@
 	(gr_poly
 		(pts
-			(xy 182.25 102.2) (xy 183.25 101.2) (xy 184.25 102.2)
+			(xy 180.78 102.49) (xy 181.78 101.49) (xy 182.78 102.49)
 		)
 		(stroke
@@
 	)
 	(gr_text "U_RX"
-		(at 185.13 105.565 270)
+		(at 186.73 105.64 270)
 		(layer "B.SilkS")
 		(effects
@@
 	)
 	(gr_text "U_TX"
-		(at 183.24 105.5 270)
+		(at 182.38 105.49 270)
 		(layer "B.SilkS")
 		(effects
