File: hardware/pawb_sao.kicad_sch (KiCad schematic)
At the start: 30 parts, among them J1 PROG, J5 SAO, Q1 MMBT3904, SW1 GREEN, SW2 RED, SW3 YELLOW, SW4 BLUE, U2 CH32V003FxPx

Commit message: made 3d model
Parts:
- SW1, SW2, SW3, SW4: footprint Button_Switch_SMD:SW_SPST_EVQP0 -> pawb_sao:SW_SPST_EVQP0
Changed lines of the file:
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@@
 			)
 		)
-		(property "Footprint" "Button_Switch_SMD:SW_SPST_EVQP0"
+		(property "Footprint" "pawb_sao:SW_SPST_EVQP0"
 			(at 208.28 113.03 0)
 			(effects
@@
 			)
 		)
-		(property "Footprint" "Button_Switch_SMD:SW_SPST_EVQP0"
+		(property "Footprint" "pawb_sao:SW_SPST_EVQP0"
 			(at 196.85 118.11 0)
 			(effects
@@
 			)
 		)
-		(property "Footprint" "Button_Switch_SMD:SW_SPST_EVQP0"
+		(property "Footprint" "pawb_sao:SW_SPST_EVQP0"
 			(at 219.71 115.57 0)
 			(effects
@@
 			)
 		)
-		(property "Footprint" "Button_Switch_SMD:SW_SPST_EVQP0"
+		(property "Footprint" "pawb_sao:SW_SPST_EVQP0"
 			(at 196.85 110.49 0)
 			(effects
